File: UI-Script/Schematics/LED_IF_circuit2.sch (EAGLE design)
At the start: 24 parts, among them Q2 BC547B, Q3 BC547B, Q4 BC547B, Q5 BC547B

Commit message: GND copper pours added
Connections:
- removed net N$7: S2.S
- net GND: now also S2.P
- net N$17: now also S2.S; no longer S2.P
Changed lines of the file:
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@@
 <label x="30.48" y="48.26" size="1.778" layer="95"/>
+</segment>
+<segment>
+<pinref part="S2" gate="1" pin="P"/>
+<wire x1="22.86" y1="-5.08" x2="22.86" y2="-10.16" width="0.1524" layer="91"/>
+<pinref part="SUPPLY6" gate="GND" pin="GND"/>
+<wire x1="22.86" y1="-10.16" x2="35.56" y2="-10.16" width="0.1524" layer="91"/>
 </segment>
 </net>
@@
 <wire x1="35.56" y1="33.02" x2="35.56" y2="7.62" width="0.1524" layer="91"/>
 <pinref part="R11" gate="G$1" pin="2"/>
-<wire x1="35.56" y1="7.62" x2="22.86" y2="7.62" width="0.1524" layer="91"/>
-<pinref part="S2" gate="1" pin="P"/>
-<wire x1="22.86" y1="7.62" x2="20.32" y2="7.62" width="0.1524" layer="91"/>
-<wire x1="22.86" y1="7.62" x2="22.86" y2="-5.08" width="0.1524" layer="91"/>
+<wire x1="35.56" y1="7.62" x2="20.32" y2="7.62" width="0.1524" layer="91"/>
+<wire x1="35.56" y1="7.62" x2="35.56" y2="-5.08" width="0.1524" layer="91"/>
+<pinref part="S2" gate="1" pin="S"/>
+<wire x1="35.56" y1="-5.08" x2="33.02" y2="-5.08" width="0.1524" layer="91"/>
 </segment>
 </net>
-<net name="N$7" class="0">
-<segment>
-<wire x1="35.56" y1="-10.16" x2="35.56" y2="-5.08" width="0.1524" layer="91"/>
-<wire x1="35.56" y1="-5.08" x2="33.02" y2="-5.08" width="0.1524" layer="91"/>
-<pinref part="S2" gate="1" pin="S"/>
-<pinref part="SUPPLY6" gate="GND" pin="GND"/>
-</segment>
-</net>

Commit message: PCB update
Parts:
- Q1: value (none) -> MMBT5088; device SparkFun-DiscreteSemi:TRANSISTOR_NPNBC547 -> SparkFun-DiscreteSemi:TRANSISTOR_NPNMMBT5088
- Q2, Q3, Q4, Q5: value BC547B -> MMBT5088; device SparkFun-DiscreteSemi:TRANSISTOR_NPNBC547 -> SparkFun-DiscreteSemi:TRANSISTOR_NPNMMBT5088
- R1, R3, R5, R7, R9: value 55 -> 1100; device SparkFun-Resistors:RESISTORPTH-1/6W -> SparkFun-Passives:RESISTOR0603-RES
- R10, R2, R4, R6, R8: value 1100 -> 55; device SparkFun-Resistors:RESISTORPTH-1/6W -> SparkFun-Passives:RESISTOR0603-RES
- R11: device SparkFun-Resistors:RESISTORPTH-1/6W -> SparkFun-Passives:RESISTOR0603-RES
Connections:
- removed net GPIO3: JP2.5, R6.1
- new net N$18: JP2.5, R5.1
- net GPIO1: now also R9.1; no longer R2.1
- net GPIO2: now also R7.1; no longer R4.1
- net GPIO4: now also R3.1; no longer R8.1
- net GPIO5: now also R1.1; no longer R10.1
- net N$10: now also R7.2; no longer R4.2
- net N$11: now also R2.2; no longer R9.2
- net N$12: now also R3.2; no longer R8.2
- net N$13: now also R4.2; no longer R7.2
- net N$14: now also R5.2; no longer R6.2
- net N$15: now also R6.2; no longer R5.2
- net N$16: now also R1.2; no longer R10.2
- net N$6: now also R10.2; no longer R1.2
- net N$8: now also R9.2; no longer R2.2
- net N$9: now also R8.2; no longer R3.2
- net VDD: now also R10.1, R2.1, R4.1, R6.1, R8.1; no longer R1.1, R3.1, R5.1, R7.1, R9.1
Other:
- moved on the sheet: R1, R10, R2, R3, R4, R5, R6, R7, R8, R9

Commit message: no error DRC
Connections:
- net N$18 renamed GPIO3
Changed lines of the file:
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@@
 </segment>
 </net>
-<net name="N$18" class="0">
+<net name="GPIO3" class="0">
 <segment>
 <pinref part="JP2" gate="A" pin="5"/>
 <wire x1="73.66" y1="40.64" x2="25.4" y2="40.64" width="0.1524" layer="91"/>
 <pinref part="R5" gate="G$1" pin="1"/>
+<label x="30.48" y="40.64" size="1.778" layer="95"/>
 </segment>
 </net>
